File: rev_a/bus_microbus2.kicad_pcb (KiCad board)
At the start: 2 copper layers, 100 x 50 mm, 40 parts, among them J1 TERMINATE_JUMPER, SW1 MJTP1243, U1 74HCT08, U2 78L05AC, U3 MCP2562, U4 L78L33AC, U5 ATMEGA328_DIP28, X1 16MHz

Commit message: Mistyped the module name.
Other:
- board text added: "BUS_MICROBUS2 REV. A 8FEB2015 (C) 2015 BY GRAMLICH"
- board text removed: "BUS_MICROBUS REV. A 8FEB2015 (C) 2015 BY GRAMLICH"
